File: Current-Meter-Eagle/draft2.brd (EAGLE design)
At the start: 50 x 50 mm, 27 parts, among them J1 USB-MICROB", J2 87520, J3 JTAG-6, J4 TFTLCDTFTLCD-DEV, U1 TPS63000DRCR, X1 CINCH-BANANA, X2 CINCH-BANANA

Commit message: Add files via upload
Routing:
- net 3.3V: track 143.3 -> 139.7 mm, vias 8 -> 6
Changed lines of the file:
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@@
 </class>
 </classes>
-<designrules name="default">
+<designrules name="SeeedStudio_2layer_DRU_no_angle_20140221">
 <description language="de">&lt;b&gt;EAGLE Design Rules&lt;/b&gt;
 &lt;p&gt;
@@
 necessary adjustments and save your customized
 design rules under a new name.</description>
+<description language="zh">&lt;b&gt;Seeed Studio EAGLE Design Rules&lt;/b&gt;
+</description>
 <param name="layerSetup" value="(1*16)"/>
-<param name="mtCopper" value="0.035mm 0.035mm 0.035mm 0.035mm 0.035mm 0.035mm 0.035mm 0.035mm 0.035mm 0.035mm 0.035mm 0.035mm 0.035mm 0.035mm 0.035mm 0.035mm"/>
-<param name="mtIsolate" value="1.5mm 0.15mm 0.2mm 0.15mm 0.2mm 0.15mm 0.2mm 0.15mm 0.2mm 0.15mm 0.2mm 0.15mm 0.2mm 0.15mm 0.2mm"/>
-<param name="mdWireWire" value="8mil"/>
-<param name="mdWirePad" value="8mil"/>
-<param name="mdWireVia" value="8mil"/>
-<param name="mdPadPad" value="8mil"/>
-<param name="mdPadVia" value="8mil"/>
-<param name="mdViaVia" value="8mil"/>
-<param name="mdSmdPad" value="8mil"/>
-<param name="mdSmdVia" value="8mil"/>
-<param name="mdSmdSmd" value="8mil"/>
+<param name="mtCopper" value="0.035mm 0.0175mm 0.035mm 0.035mm 0.035mm 0.035mm 0.035mm 0.035mm 0.035mm 0.035mm 0.035mm 0.035mm 0.035mm 0.035mm 0.0175mm 0.035mm"/>
+<param name="mtIsolate" value="1.5mm 1.1mm 0.2mm 0.15mm 0.2mm 0.15mm 0.2mm 0.15mm 0.2mm 0.15mm 0.2mm 0.15mm 0.2mm 0.15mm 0.2mm"/>
+<param name="mdWireWire" value="6mil"/>
+<param name="mdWirePad" value="6mil"/>
+<param name="mdWireVia" value="6mil"/>
+<param name="mdPadPad" value="6mil"/>
+<param name="mdPadVia" value="6mil"/>
+<param name="mdViaVia" value="6mil"/>
+<param name="mdSmdPad" value="0mil"/>
+<param name="mdSmdVia" value="0mil"/>
+<param name="mdSmdSmd" value="0mil"/>
 <param name="mdViaViaSameLayer" value="8mil"/>
 <param name="mnLayersViaInSmd" value="2"/>
-<param name="mdCopperDimension" value="40mil"/>
-<param name="mdDrill" value="8mil"/>
+<param name="mdCopperDimension" value="10mil"/>
+<param name="mdDrill" value="10mil"/>
 <param name="mdSmdStop" value="0mil"/>
-<param name="msWidth" value="10mil"/>
-<param name="msDrill" value="24mil"/>
-<param name="msMicroVia" value="9.99mm"/>
+<param name="msWidth" value="6mil"/>
+<param name="msDrill" value="12mil"/>
+<param name="msMicroVia" value="12mil"/>
 <param name="msBlindViaRatio" value="0.5"/>
 <param name="rvPadTop" value="0.25"/>
@@
 <param name="rlMinPadBottom" value="10mil"/>
 <param name="rlMaxPadBottom" value="20mil"/>
-<param name="rlMinViaOuter" value="8mil"/>
+<param name="rlMinViaOuter" value="6mil"/>
 <param name="rlMaxViaOuter" value="20mil"/>
-<param name="rlMinViaInner" value="8mil"/>
+<param name="rlMinViaInner" value="6mil"/>
 <param name="rlMaxViaInner" value="20mil"/>
 <param name="rlMinMicroViaOuter" value="4mil"/>
@@
 <param name="psTop" value="-1"/>
 <param name="psBottom" value="-1"/>
-<param name="psFirst" value="-1"/>
+<param name="psFirst" value="0"/>
 <param name="psElongationLong" value="100"/>
 <param name="psElongationOffset" value="100"/>
 <param name="mvStopFrame" value="1"/>
 <param name="mvCreamFrame" value="0"/>
-<param name="mlMinStopFrame" value="4mil"/>
-<param name="mlMaxStopFrame" value="4mil"/>
+<param name="mlMinStopFrame" value="2mil"/>
+<param name="mlMaxStopFrame" value="2mil"/>
 <param name="mlMinCreamFrame" value="0mil"/>
 <param name="mlMaxCreamFrame" value="0mil"/>
-<param name="mlViaStopLimit" value="0mil"/>
+<param name="mlViaStopLimit" value="100mil"/>
 <param name="srRoundness" value="0"/>
 <param name="srMinRoundness" value="0mil"/>
@@
 <param name="checkAngle" value="0"/>
 <param name="checkFont" value="1"/>
-<param name="checkRestrict" value="1"/>
+<param name="checkRestrict" value="0"/>
 <param name="useDiameter" value="13"/>
 <param name="maxErrors" value="50"/>
@@
 <element name="J3" library="00ese323" package="JTAG6" value="JTAG-6" x="92" y="44.75" rot="R270"/>
 <element name="J4" library="00ese323" package="TFTLCD" value="TFTLCDTFTLCD-DEV" x="100.16" y="32.96"/>
-<element name="PB1" library="00ese323" package="PB-B3FS-1010P" value="PB-B3FS-1010P" x="56.99" y="18.52" rot="R90"/>
-<element name="PB2" library="00ese323" package="PB-B3FS-1010P" value="PB-B3FS-1010P" x="56.99" y="30.92" rot="R90"/>
+<element name="PB1" library="00ese323" package="PB-B3FS-1010P" value="PB-B3FS-1010P" x="56.99" y="18.52" smashed="yes" rot="R90">
+<attribute name="NAME" x="53.69" y="17.02" size="1.27" layer="25" rot="R90"/>
+</element>
+<element name="PB2" library="00ese323" package="PB-B3FS-1010P" value="PB-B3FS-1010P" x="56.99" y="30.92" smashed="yes" rot="R90">
+<attribute name="NAME" x="53.69" y="29.62" size="1.27" layer="25" rot="R90"/>
+</element>
 <element name="R1" library="00ese323" package="RC1206" value="1k" x="87.73" y="36.13"/>
 <element name="R10" library="00ese323" package="0402" value="CRCW04021M00FKED" x="63.07" y="48.18">
@@
 <via x="61.625" y="47.5" extent="1-16" drill="0.6096"/>
 <via x="67.625" y="46.625" extent="1-16" drill="0.6096"/>
-<wire x1="75.4274" y1="24.49" x2="71.31" y2="24.49" width="0.254" layer="1"/>
-<wire x1="71.31" y1="24.49" x2="67.3" y2="28.5" width="0.254" layer="1"/>
-<via x="67.3" y="28.5" extent="1-16" drill="0.6"/>
-<wire x1="67.3" y1="28.5" x2="64.7" y2="31.1" width="0.254" layer="16"/>
-<via x="64.7" y="31.1" extent="1-16" drill="0.6"/>
-<wire x1="64.7" y1="31.1" x2="63.42" y2="31.1" width="0.254" layer="1"/>
-<wire x1="63.42" y1="31.1" x2="59.24" y2="26.92" width="0.254" layer="1"/>
 <wire x1="59.24" y1="26.92" x2="59.24" y2="26.84" width="0.254" layer="1"/>
-<wire x1="59.24" y1="26.84" x2="57.3" y2="24.9" width="0.254" layer="1"/>
-<via x="57.3" y="24.9" extent="1-16" drill="0.6"/>
-<wire x1="57.3" y1="24.9" x2="57.3" y2="18.6" width="0.254" layer="16"/>
-<via x="57.3" y="18.6" extent="1-16" drill="0.6"/>
-<wire x1="57.3" y1="18.6" x2="57.3" y2="16.46" width="0.254" layer="1"/>
-<wire x1="57.3" y1="16.46" x2="59.24" y2="14.52" width="0.254" layer="1"/>
+<wire x1="59.24" y1="26.84" x2="61.56" y2="26.84" width="0.254" layer="1"/>
+<wire x1="61.56" y1="26.84" x2="61.6" y2="26.8" width="0.254" layer="1"/>
+<via x="61.6" y="26.8" extent="1-16" drill="0.6"/>
+<wire x1="61.6" y1="26.8" x2="61.6" y2="25.4" width="0.254" layer="16"/>
+<wire x1="61.6" y1="25.4" x2="62.4" y2="24.6" width="0.254" layer="16"/>
+<via x="62.4" y="24.6" extent="1-16" drill="0.6"/>
+<wire x1="62.4" y1="24.6" x2="75.3174" y2="24.6" width="0.254" layer="1"/>
+<wire x1="75.3174" y1="24.6" x2="75.4274" y2="24.49" width="0.254" layer="1"/>
+<wire x1="62.4" y1="24.6" x2="62.4" y2="15.1" width="0.254" layer="1"/>
+<wire x1="62.4" y1="15.1" x2="61.6" y2="14.3" width="0.254" layer="1"/>
+<wire x1="61.6" y1="14.3" x2="59.46" y2="14.3" width="0.254" layer="1"/>
+<wire x1="59.46" y1="14.3" x2="59.24" y2="14.52" width="0.254" layer="1"/>
 </signal>
 <signal name="3V">
