File: Current-Meter-Eagle/mtsch.brd (EAGLE design)
At the start: 160 x 100 mm, 7 parts, among them IC1 AD8541R

Commit message: Add files via upload
Parts:
- moved C1 37.0 mm to (21.6, 27.9)
Routing:
- net N$3: track 41.8 -> 44.5 mm
- net GND: track 68.7 -> 67.8 mm
- net N$1: track 21.0 -> 21.5 mm
Other:
- board size 160 x 100 mm -> 36.8 x 37.8 mm
- board text added: ">Frank Yee 109374525"
Changed lines of the file:
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@@
 <board>
 <plain>
-<wire x1="0" y1="0" x2="160" y2="0" width="0" layer="20"/>
-<wire x1="160" y1="0" x2="160" y2="100" width="0" layer="20"/>
-<wire x1="160" y1="100" x2="0" y2="100" width="0" layer="20"/>
-<wire x1="0" y1="100" x2="0" y2="0" width="0" layer="20"/>
+<wire x1="0" y1="0" x2="36.81" y2="0" width="0" layer="20"/>
+<wire x1="36.81" y1="0" x2="36.81" y2="37.77" width="0" layer="20"/>
+<wire x1="36.81" y1="37.77" x2="0" y2="37.77" width="0" layer="20"/>
+<wire x1="0" y1="37.77" x2="0" y2="0" width="0" layer="20"/>
+<text x="2.54" y="33.02" size="1.778" layer="21">&gt;Frank Yee 109374525</text>
 </plain>
 <attributes>
@@
 <attribute name="OC_NEWARK" value="27C1933" x="11.43" y="17.78" size="1.778" layer="27" rot="R90" display="off"/>
 </element>
-<element name="C1" library="resistor" package="C3216" value="1u" x="2.54" y="-3.81"/>
+<element name="C1" library="resistor" package="C3216" value="1u" x="21.59" y="27.94"/>
 </elements>
 <signals>
@@
 <contactref element="X1" pad="5"/>
 <contactref element="IC1" pad="7"/>
-<wire x1="12.065" y1="21.59" x2="13.335" y2="22.86" width="0.254" layer="1"/>
-<wire x1="13.335" y1="22.86" x2="18.415" y2="27.94" width="0.254" layer="1"/>
-<wire x1="11.43" y1="21.59" x2="12.065" y2="21.59" width="0.254" layer="1"/>
+<contactref element="C1" pad="1"/>
+<wire x1="13.335" y1="21.59" x2="19.685" y2="27.94" width="0.254" layer="1"/>
+<wire x1="11.43" y1="21.59" x2="13.335" y2="21.59" width="0.254" layer="1"/>
+<wire x1="19.685" y1="27.94" x2="20.19" y2="27.94" width="0.254" layer="1"/>
 <wire x1="13.335" y1="18.415" x2="20.26" y2="18.415" width="0.254" layer="1"/>
-<wire x1="13.335" y1="22.86" x2="13.335" y2="18.415" width="0.254" layer="1"/>
-<contactref element="C1" pad="1"/>
-<wire x1="1.14" y1="-3.81" x2="13.335" y2="18.415" width="0" layer="19" extent="1-1"/>
+<wire x1="13.335" y1="21.59" x2="13.335" y2="18.415" width="0.254" layer="1"/>
 </signal>
 <signal name="GND">
@@
 <contactref element="TP1" pad="GND"/>
 <contactref element="TP2" pad="GND"/>
-<wire x1="25.4" y1="24.765" x2="24.13" y2="26.035" width="0.254" layer="1"/>
-<wire x1="24.13" y1="26.035" x2="22.225" y2="27.94" width="0.254" layer="1"/>
-<wire x1="25.4" y1="20.955" x2="25.4" y2="24.765" width="0.254" layer="1"/>
+<contactref element="C1" pad="2"/>
+<wire x1="25.4" y1="26.035" x2="24.765" y2="26.67" width="0.254" layer="1"/>
+<wire x1="24.765" y1="26.67" x2="23.495" y2="27.94" width="0.254" layer="1"/>
+<wire x1="25.4" y1="20.955" x2="25.4" y2="26.035" width="0.254" layer="1"/>
+<wire x1="23.495" y1="27.94" x2="22.99" y2="27.94" width="0.254" layer="1"/>
 <wire x1="25.4" y1="20.955" x2="25.46" y2="20.955" width="0.254" layer="1"/>
 <wire x1="33.02" y1="25.4" x2="30.48" y2="27.94" width="0.254" layer="1"/>
 <wire x1="33.02" y1="22.05" x2="33.02" y2="25.4" width="0.254" layer="1"/>
 <wire x1="30.48" y1="27.94" x2="30.16" y2="27.94" width="0.254" layer="1"/>
+<wire x1="27.305" y1="29.21" x2="24.765" y2="26.67" width="0.254" layer="1"/>
+<wire x1="29.845" y1="29.21" x2="27.305" y2="29.21" width="0.254" layer="1"/>
+<wire x1="29.845" y1="27.94" x2="29.845" y2="29.21" width="0.254" layer="1"/>
+<wire x1="29.845" y1="27.94" x2="30.16" y2="27.94" width="0.254" layer="1"/>
 <wire x1="13.335" y1="15.875" x2="11.43" y2="13.97" width="0.254" layer="1"/>
 <wire x1="13.335" y1="17.145" x2="13.335" y2="15.875" width="0.254" layer="1"/>
@@
 <wire x1="11.43" y1="24.13" x2="31.115" y2="24.13" width="0.254" layer="16"/>
 <wire x1="33.02" y1="22.225" x2="33.02" y2="22.05" width="0.254" layer="16"/>
-<wire x1="27.305" y1="29.21" x2="24.13" y2="26.035" width="0.254" layer="1"/>
-<wire x1="29.845" y1="29.21" x2="27.305" y2="29.21" width="0.254" layer="1"/>
-<wire x1="29.845" y1="27.94" x2="29.845" y2="29.21" width="0.254" layer="1"/>
-<wire x1="29.845" y1="27.94" x2="30.16" y2="27.94" width="0.254" layer="1"/>
-<contactref element="C1" pad="2"/>
-<wire x1="3.94" y1="-3.81" x2="11.43" y2="13.97" width="0" layer="19" extent="1-1"/>
 </signal>
 <signal name="N$3">
@@
 <wire x1="22.86" y1="19.685" x2="25.46" y2="19.685" width="0.254" layer="1"/>
 <wire x1="22.86" y1="16.51" x2="22.86" y2="19.685" width="0.254" layer="1"/>
-<wire x1="16.51" y1="10.16" x2="22.86" y2="16.51" width="0.254" layer="1"/>
-<wire x1="3.81" y1="10.16" x2="9.525" y2="10.16" width="0.254" layer="1"/>
-<wire x1="9.525" y1="10.16" x2="16.51" y2="10.16" width="0.254" layer="1"/>
-<wire x1="3.81" y1="17.32" x2="3.81" y2="10.16" width="0.254" layer="1"/>
+<wire x1="16.51" y1="8.89" x2="22.86" y2="16.51" width="0.254" layer="1"/>
+<wire x1="9.525" y1="8.89" x2="16.51" y2="8.89" width="0.254" layer="1"/>
 <wire x1="9.525" y1="14.605" x2="11.43" y2="16.51" width="0.254" layer="1"/>
-<wire x1="9.525" y1="10.16" x2="9.525" y2="14.605" width="0.254" layer="1"/>
+<wire x1="9.525" y1="8.89" x2="9.525" y2="14.605" width="0.254" layer="1"/>
+<wire x1="9.525" y1="8.89" x2="5.08" y2="8.89" width="0.254" layer="1"/>
+<wire x1="5.08" y1="8.89" x2="3.81" y2="10.16" width="0.254" layer="1"/>
+<wire x1="3.81" y1="10.16" x2="3.81" y2="17.32" width="0.254" layer="1"/>
 </signal>
 <signal name="N$5">
